Commit message: fix(physics): boost steering effort/gains and WheelSlip compliance for Featherstone
Steering joints: effort 100→500 Nm, p_gain 50→500, i_gain 0.1→0.5, d_gain 1→5
WheelSlip front wheels: lateral 0.005→0.15, longitudinal 0.005→0.12
Required after Bullet Featherstone migration (01e4166) which ignores legacy
<gazebo reference> slip tags, leaving servos unable to overcome rigid friction.

File: src/2_ugv_fleet_brain/bot_description/urdf/bot.urdf.xacro (robot description, xacro)
@@ -78,5 +78,5 @@
     <child link="base_front_left_steering"/>
     <origin xyz="0.39 -0.265 -0.2075" rpy="-1.57079632679 0 0"/>
-    <limit lower="-0.2616" upper="0.2616" effort="100" velocity="1.0"/>
+    <limit lower="-0.2616" upper="0.2616" effort="500" velocity="1.0"/>
     <axis xyz="0 1 0"/>
   </joint>
@@ -107,5 +107,5 @@
     <child link="base_front_right_steering"/>
     <origin xyz="0.39 0.265 -0.2075" rpy="-1.57079632679 0 0"/>
-    <limit lower="-0.2616" upper="0.2616" effort="100" velocity="1.0"/>
+    <limit lower="-0.2616" upper="0.2616" effort="500" velocity="1.0"/>
     <axis xyz="0 1 0"/>
   </joint>
@@ -684,14 +684,14 @@
       <joint_name>base_front_left_steering_joint</joint_name>
       <topic>/model/$(arg bot_name)/joint/base_front_left_steering_joint/cmd_pos</topic>
-      <p_gain>50.0</p_gain>
-      <i_gain>0.1</i_gain>
-      <d_gain>1.0</d_gain>
+      <p_gain>500.0</p_gain>
+      <i_gain>0.5</i_gain>
+      <d_gain>5.0</d_gain>
     </plugin>
     <plugin filename="gz-sim-joint-position-controller-system" name="gz::sim::systems::JointPositionController">
       <joint_name>base_front_right_steering_joint</joint_name>
       <topic>/model/$(arg bot_name)/joint/base_front_right_steering_joint/cmd_pos</topic>
-      <p_gain>50.0</p_gain>
-      <i_gain>0.1</i_gain>
-      <d_gain>1.0</d_gain>
+      <p_gain>500.0</p_gain>
+      <i_gain>0.5</i_gain>
+      <d_gain>5.0</d_gain>
     </plugin>
     <plugin filename="gz-sim-joint-controller-system" name="gz::sim::systems::JointController">
@@ -758,12 +758,12 @@
     <plugin filename="gz-sim-wheel-slip-system" name="gz::sim::systems::WheelSlip">
       <wheel link_name="base_front_left_wheel">
-        <slip_compliance_lateral>0.005</slip_compliance_lateral>
-        <slip_compliance_longitudinal>0.005</slip_compliance_longitudinal>
+        <slip_compliance_lateral>0.15</slip_compliance_lateral>
+        <slip_compliance_longitudinal>0.12</slip_compliance_longitudinal>
         <wheel_normal_force>43</wheel_normal_force>
         <wheel_radius>0.175</wheel_radius>
       </wheel>
       <wheel link_name="base_front_right_wheel">
-        <slip_compliance_lateral>0.005</slip_compliance_lateral>
-        <slip_compliance_longitudinal>0.005</slip_compliance_longitudinal>
+        <slip_compliance_lateral>0.15</slip_compliance_lateral>
+        <slip_compliance_longitudinal>0.12</slip_compliance_longitudinal>
         <wheel_normal_force>43</wheel_normal_force>
         <wheel_radius>0.175</wheel_radius>

Commit message: revert(physics): restore dartsim+ODE engine, revert Featherstone URDF tuning
Reverts commit 01e4166 (Featherstone engine switch) and 44d3e0f (steering
gain boost). dartsim+ODE correctly parses legacy <gazebo reference> slip
tags and the original steering effort/gains work fine with it. Featherstone
introduced steering jams and unpredictable behavior that isn't worth the
migration effort for a 16 kg desert UGV.

File: src/2_ugv_fleet_brain/bot_description/urdf/bot.urdf.xacro (robot description, xacro)
@@ -78,5 +78,5 @@
     <child link="base_front_left_steering"/>
     <origin xyz="0.39 -0.265 -0.2075" rpy="-1.57079632679 0 0"/>
-    <limit lower="-0.2616" upper="0.2616" effort="500" velocity="1.0"/>
+    <limit lower="-0.2616" upper="0.2616" effort="100" velocity="1.0"/>
     <axis xyz="0 1 0"/>
   </joint>
@@ -107,5 +107,5 @@
     <child link="base_front_right_steering"/>
     <origin xyz="0.39 0.265 -0.2075" rpy="-1.57079632679 0 0"/>
-    <limit lower="-0.2616" upper="0.2616" effort="500" velocity="1.0"/>
+    <limit lower="-0.2616" upper="0.2616" effort="100" velocity="1.0"/>
     <axis xyz="0 1 0"/>
   </joint>
@@ -684,14 +684,14 @@
       <joint_name>base_front_left_steering_joint</joint_name>
       <topic>/model/$(arg bot_name)/joint/base_front_left_steering_joint/cmd_pos</topic>
-      <p_gain>500.0</p_gain>
-      <i_gain>0.5</i_gain>
-      <d_gain>5.0</d_gain>
+      <p_gain>50.0</p_gain>
+      <i_gain>0.1</i_gain>
+      <d_gain>1.0</d_gain>
     </plugin>
     <plugin filename="gz-sim-joint-position-controller-system" name="gz::sim::systems::JointPositionController">
       <joint_name>base_front_right_steering_joint</joint_name>
       <topic>/model/$(arg bot_name)/joint/base_front_right_steering_joint/cmd_pos</topic>
-      <p_gain>500.0</p_gain>
-      <i_gain>0.5</i_gain>
-      <d_gain>5.0</d_gain>
+      <p_gain>50.0</p_gain>
+      <i_gain>0.1</i_gain>
+      <d_gain>1.0</d_gain>
     </plugin>
     <plugin filename="gz-sim-joint-controller-system" name="gz::sim::systems::JointController">
@@ -758,12 +758,12 @@
     <plugin filename="gz-sim-wheel-slip-system" name="gz::sim::systems::WheelSlip">
       <wheel link_name="base_front_left_wheel">
-        <slip_compliance_lateral>0.15</slip_compliance_lateral>
-        <slip_compliance_longitudinal>0.12</slip_compliance_longitudinal>
+        <slip_compliance_lateral>0.005</slip_compliance_lateral>
+        <slip_compliance_longitudinal>0.005</slip_compliance_longitudinal>
         <wheel_normal_force>43</wheel_normal_force>
         <wheel_radius>0.175</wheel_radius>
       </wheel>
       <wheel link_name="base_front_right_wheel">
-        <slip_compliance_lateral>0.15</slip_compliance_lateral>
-        <slip_compliance_longitudinal>0.12</slip_compliance_longitudinal>
+        <slip_compliance_lateral>0.005</slip_compliance_lateral>
+        <slip_compliance_longitudinal>0.005</slip_compliance_longitudinal>
         <wheel_normal_force>43</wheel_normal_force>
         <wheel_radius>0.175</wheel_radius>
